Commit message: corrected angles in urdf file, moved urdf file over to other places temporarily (I am going to redo the entire codebase stucture...eventually)

File: urdf/lekiwi/LeKiwi.urdf (robot description, URDF)
Before this commit: robot LeKiwi, 45 links, 44 joints
Joints:
- joint STS3215_03a-v1-1_Revolute-49: limit (none) -> lower=2.96547 upper=6.45772 effort=10 velocity=10; type continuous -> revolute
- joint STS3215_03a-v1-2_Revolute-51: limit (none) -> lower=-0.17453 upper=3.14159 effort=10 velocity=10; type continuous -> revolute
- joint STS3215_03a-v1-3_Revolute-53: limit (none) -> lower=-0.08727 upper=3.22885 effort=10 velocity=10; type continuous -> revolute
- joint STS3215_03a-v1-4_Revolute-57: limit (none) -> lower=4.71079632679 upper=6.45771632679 effort=10 velocity=10; type continuous -> revolute
- joint STS3215_03a-v1_Revolute-45: limit (none) -> lower=4.36173 upper=8.20145 effort=10 velocity=10; type continuous -> revolute
- joint STS3215_03a_Wrist_Roll-v1_Revolute-55: limit (none) -> lower=0.39774 upper=5.9828 effort=10 velocity=10; type continuous -> revolute
